Commit message: removed last reference to old project

File: qlab/qlab_description/urdf/sensors/sonar_sensor.urdf.xacro (robot description, xacro)
@@ -20,5 +20,5 @@
         <geometry>
           <!--<box size="0.01 0.01 0.01" /> -->
-          <mesh filename="package://ardrone_vislab_description/meshes/sonar_sensor/max_sonar_ez4.dae"/>
+          <mesh filename="package://qlab_description/meshes/sonar_sensor/max_sonar_ez4.dae"/>
         </geometry>
       </visual>
