Commit message: Kingfisher files added

File: qlab/qlab_description/urdf/sensors/hokuyo_utm30lx.urdf.xacro (robot description, xacro)
@@ -19,5 +19,5 @@
 	  <origin xyz="0 0 0" rpy="0 0 0" />
           <geometry>
-          <mesh filename="package://ardrone_vislab_description/meshes/hokuyo_utm30lx/hokuyo_utm_30lx$(optenv TEST_SELF_FILTER).dae"/>
+          <mesh filename="package://qlab_description/meshes/hokuyo_utm30lx/hokuyo_utm_30lx$(optenv TEST_SELF_FILTER).dae"/>
         </geometry>
 	</visual>
